File: ProFinalKicadV1.sch (KiCad schematic (older format))
At the start: 22 parts, among them SW501 SPST, U1 MICRO-B_USB, U2 MIC5219-3.3BM5, U3 FT231XS, U4 XB24-Z7WIT-004

Commit message: Actualizando Esquematico Rev 1.3 y campos Kicost
Actualizando Esquematico en base a a la Rev 1.3 y campos Kicost
faltantes
Parts:
- added P1, P2: CONN_01X02, symbol CONN_01X02
- C1, R1, R2, R6: Digikey# (none) -> MCT0603-1.00K-CFTR-ND; Manf (none) -> Vishay Beyschlag; Manf# (none) -> MCT06030C1001FP500
- C2, C3: Digikey# (none) -> 445-1277-1-ND; Manf (none) -> TDK Corporation; Manf# (none) -> C1608C0G1H470J080AA
- C4, C6: Digikey# (none) -> 311-1343-1-ND; Manf (none) -> Yageo; Manf# (none) -> CC0603ZRY5V9BB104
- C5: Digikey# (none) -> 493-14027-2-ND; Manf (none) -> Nichicon; Manf# (none) -> PCF1E100MCL1GS
- D1, D3: Digikey# (none) -> 475-2920-1-ND; Manf (none) -> OSRAM Opto Semiconductors Inc.; Manf# (none) -> LP L296-J2L2-25-Z
- D2, D4: Digikey# (none) -> 475-2512-1-ND; Manf (none) -> OSRAM Opto Semiconductors Inc.; Manf# (none) -> LS Q976-NR-1
- R3, R4: Digikey# (none) -> P27GCT-ND; MF Panasonic -> (none); MP ERJ-3GEYJ270V -> (none); Manf (none) -> Panasonic Electronic Components; Manf# (none) -> ERJ-3GEYJ270V; Price 0.01 USD -> (none)
- SW501, XA1: Digikey# (none) -> 952-1938-ND; Manf (none) -> Harwin Inc.; Manf# (none) -> D01-9973242
- U1: Digikey# (none) -> 732-2734-ND; Manf (none) -> Wurth Electronics Inc.; Manf# (none) -> 61400413321
- U2: Digikey# (none) -> MIC5219-3.3BM5-TR-ND; Manf (none) -> Microchip Technology; Manf# (none) -> MIC5219-3.3BM5-TR
- U3: Digikey# (none) -> 768-1129-1-ND; MF FTDI -> (none); MP FT231XS -> (none); MP_odl (none) -> FT231XS; Manf (none) -> FTDI, Future Technology Devices International Ltd; Manf# (none) -> FT231XS-R; Price 2.63 USD -> (none); Price_aprox (none) -> 2.63 USD
- U4: Digikey# (none) -> 602-1098-ND; MF Digi International -> (none); MP XB24-Z7WIT-004 -> (none); Manf (none) -> Digi International; Manf# (none) -> XB24-Z7WIT-004; Price None -> (none)
Connections:
- net +3V3: now also P2.2 (P2); no longer U2.5 (OUT)
- net +5V: now also P1.1 (P1); no longer U2.1 (VIN)
- net CTS_XBEE: no longer names the net of U3.P6 (CTS#), U4.12
- net DTR_XBEE renamed DTS_DTR_XBEE
- net RTS_XBEE: no longer names the net of U3.P19 (RTS#), U4.16
- new net: P1.2 (P2), U2.1 (VIN)
- new net: P2.1 (P1), U2.5 (OUT)
Other:
- note added: "P1 y P2 se colocan para el uso del poncho\nsin la EDU-CIAA-NXP.\nSe alimentara por USB y se debera unir los \npines 1 y 2 de P1 \ny los pines 1 y 2 de P2."
- note removed: "Aclaracion\nEl pin (18) DTR# en FT231XS es DTS_XBEE \nes la misma coneccion del pin (9) DTR_XBEE\nen Xbee"
- moved on the sheet: C5, C6, D3, R5, SW501, U4

Commit message: Asociando 3D
3D de elementos previo a ruteo de PCB
Parts:
- C1, C4, C6: footprint Capacitors_SMD:C_0603_HandSoldering -> C_0_1uF_pretty:C_0603_HandSoldering
- C2, C3: footprint Capacitors_SMD:C_0603_HandSoldering -> C_47pF_pretty:C_0603_HandSoldering
- C5: footprint Capacitors_SMD:CP_Elec_8x10 -> C_10uF_pretty:CP_4x5mm
- P1, P2: footprint (none) -> w_pin_strip.pretty:pin_socket_2
- R3, R4: footprint RESC1608X55 -> R_27Ohm_pretty:r_0603
- SW501: footprint Measurement_Points:Test_Point_2Pads -> Switch_pretty:smd_push
- U1: footprint Connect:USB_B -> USB_pretty:conn_usb_B_micro_smd
- U2: footprint TO_SOT_Packages_SMD:TSOT-23-5_HandSoldering -> MIC5219-3.3BM5_pretty:sot23-5
- U3: footprint RF_Modules:Digi_XBee_SMT -> FT231XS_pretty:qfn-20
- U4: footprint Housings_SOIC:SOIC-20W_7.5x12.8mm_Pitch1.27mm -> Xbee_pretty:XBee
Changed lines of the file:
@@
 F 0 "U3" H 5050 2350 50  0000 L BNN
 F 1 "FT231XS" H 4950 2450 50  0000 L BNN
-F 2 "RF_Modules:Digi_XBee_SMT" H 4800 3550 50  0001 L BNN
+F 2 "FT231XS_pretty:qfn-20" H 4800 3550 50  0001 L BNN
 F 3 "SSOP-20 FTDI" H 4800 3450 50  0001 L BNN
 F 4 "FT231XS" H 4800 3350 50  0001 L BNN "MP_odl"
@@
 F 0 "C4" H 3325 2000 50  0000 L CNN
 F 1 "0.1uF" H 3325 1800 50  0000 L CNN
-F 2 "Capacitors_SMD:C_0603_HandSoldering" H 3338 1750 50  0001 C CNN
+F 2 "C_0_1uF_pretty:C_0603_HandSoldering" H 3338 1750 50  0001 C CNN
 F 3 "" H 3300 1900 50  0000 C CNN
 F 4 "311-1343-1-ND" H 3300 1900 60  0001 C CNN "Digikey#"
@@
 F 0 "C1" H 9775 4700 50  0000 L CNN
 F 1 "0.1uF" H 9775 4500 50  0000 L CNN
-F 2 "Capacitors_SMD:C_0603_HandSoldering" H 9788 4450 50  0001 C CNN
+F 2 "C_0_1uF_pretty:C_0603_HandSoldering" H 9788 4450 50  0001 C CNN
 F 3 "" H 9750 4600 50  0000 C CNN
 F 4 "MCT0603-1.00K-CFTR-ND" H 9750 4600 60  0001 C CNN "Digikey#"
@@
 F 0 "C2" H 3125 2900 50  0000 L CNN
 F 1 "47pF" H 2900 2700 50  0000 L CNN
-F 2 "Capacitors_SMD:C_0603_HandSoldering" H 3138 2650 50  0001 C CNN
+F 2 "C_47pF_pretty:C_0603_HandSoldering" H 3138 2650 50  0001 C CNN
 F 3 "" H 3100 2800 50  0000 C CNN
 F 4 "445-1277-1-ND" H 3100 2800 60  0001 C CNN "Digikey#"
@@
 F 0 "C3" H 3375 2900 50  0000 L CNN
 F 1 "47pF" H 3375 2700 50  0000 L CNN
-F 2 "Capacitors_SMD:C_0603_HandSoldering" H 3388 2650 50  0001 C CNN
+F 2 "C_47pF_pretty:C_0603_HandSoldering" H 3388 2650 50  0001 C CNN
 F 3 "" H 3350 2800 50  0000 C CNN
 F 4 "445-1277-1-ND" H 3350 2800 60  0001 C CNN "Digikey#"
@@
 F 0 "R4" H 3550 2550 50  0000 L BNN
 F 1 "27" H 3750 2550 50  0000 L BNN
-F 2 "RESC1608X55" H 3700 2650 50  0001 L BNN
+F 2 "R_27Ohm_pretty:r_0603" H 3700 2650 50  0001 L BNN
 F 3 "0603 Panasonic" H 3700 2650 50  0001 L BNN
 F 4 "Resistor Thick Film 0603 27 Ohm 5%25 1/10 Watt %C2%B1200ppm %C2%B0C Surface Mount Punched Carrier Tape and Reel" H 3700 2650 50  0001 L BNN "Description"
@@
 F 0 "R3" H 3550 2509 50  0000 L BNN
 F 1 "27" H 3700 2500 50  0000 L BNN
-F 2 "RESC1608X55" H 3700 2450 50  0001 L BNN
+F 2 "R_27Ohm_pretty:r_0603" H 3700 2450 50  0001 L BNN
 F 3 "0603 Panasonic" H 3700 2450 50  0001 L BNN
 F 4 "Resistor Thick Film 0603 27 Ohm 5%25 1/10 Watt %C2%B1200ppm %C2%B0C Surface Mount Punched Carrier Tape and Reel" H 3700 2450 50  0001 L BNN "Description"
@@
 F 0 "U1" H 8650 4150 50  0000 C CNN
 F 1 "MICRO-B_USB" H 8650 4750 50  0000 C CNN
-F 2 "Connect:USB_B" H 8650 4450 60  0001 C CNN
+F 2 "USB_pretty:conn_usb_B_micro_smd" H 8650 4450 60  0001 C CNN
 F 3 "" H 8650 4450 60  0000 C CNN
 F 4 "732-2734-ND" H 8650 4450 60  0001 C CNN "Digikey#"
@@
 F 0 "U2" H 5700 5150 60  0000 C CNN
 F 1 "MIC5219-3.3BM5" H 5750 4350 60  0000 C CNN
-F 2 "TO_SOT_Packages_SMD:TSOT-23-5_HandSoldering" H 5700 4750 60  0001 C CNN
+F 2 "MIC5219-3.3BM5_pretty:sot23-5" H 5700 4750 60  0001 C CNN
 F 3 "" H 5700 4750 60  0000 C CNN
 F 4 "MIC5219-3.3BM5-TR-ND" H 5700 4750 60  0001 C CNN "Digikey#"
@@
 F 0 "C5" H 6625 4800 50  0000 L CNN
 F 1 "10uF" H 6625 4600 50  0000 L CNN
-F 2 "Capacitors_SMD:CP_Elec_8x10" H 6600 4700 50  0001 C CNN
+F 2 "C_10uF_pretty:CP_4x5mm" H 6600 4700 50  0001 C CNN
 F 3 "" H 6600 4700 50  0000 C CNN
 F 4 "493-14027-2-ND" H 6600 4700 60  0001 C CNN "Digikey#"
@@
 F 0 "C6" H 6925 4800 50  0000 L CNN
 F 1 "0.1uF" H 6925 4600 50  0000 L CNN
-F 2 "Capacitors_SMD:C_0603_HandSoldering" H 6938 4550 50  0001 C CNN
+F 2 "C_0_1uF_pretty:C_0603_HandSoldering" H 6938 4550 50  0001 C CNN
 F 3 "" H 6900 4700 50  0000 C CNN
 F 4 "311-1343-1-ND" H 6900 4700 60  0001 C CNN "Digikey#"
@@
 F 0 "SW501" H 10650 3300 50  0000 C CNN
 F 1 "SPST" H 10650 3100 50  0000 C CNN
-F 2 "Measurement_Points:Test_Point_2Pads" H 10650 3200 50  0001 C CNN
+F 2 "Switch_pretty:smd_push" H 10650 3200 50  0001 C CNN
 F 3 "" H 10650 3200 50  0000 C CNN
 F 4 "952-1938-ND" H 10650 3200 60  0001 C CNN "Digikey#"
@@
 F 0 "U4" H 8800 3100 50  0000 L BNN
 F 1 "XB24-Z7WIT-004" H 8850 2700 50  0001 L BNN
-F 2 "Housings_SOIC:SOIC-20W_7.5x12.8mm_Pitch1.27mm" H 8850 2700 50  0001 L BNN
+F 2 "Xbee_pretty:XBee" H 8850 2700 50  0001 L BNN
 F 3 "DIP-20 Digi International" H 8850 2700 50  0001 L BNN
 F 4 "Xbee Zb %28Zigbee Pro Feature Set%29%2C 1mw%2C Wire Antenna%2C 250000" H 8850 2700 50  0001 L BNN "Description"
@@
 F 0 "P1" H 4750 4500 50  0000 C CNN
 F 1 "CONN_01X02" V 4850 4350 50  0000 C CNN
-F 2 "" H 4750 4350 50  0000 C CNN
+F 2 "w_pin_strip.pretty:pin_socket_2" H 4750 4350 50  0001 C CNN
 F 3 "" H 4750 4350 50  0000 C CNN
 F 4 "952-1938-ND" H 4750 4350 60  0001 C CNN "Digikey#"
@@
 F 0 "P2" H 6350 4500 50  0000 C CNN
 F 1 "CONN_01X02" V 6450 4350 50  0000 C CNN
-F 2 "" H 6350 4350 50  0000 C CNN
+F 2 "w_pin_strip.pretty:pin_socket_2" H 6350 4350 50  0001 C CNN
 F 3 "" H 6350 4350 50  0000 C CNN
 F 4 "952-1938-ND" H 6350 4350 60  0001 C CNN "Digikey#"

Commit message: PCB
Ruteo de la placa
Parts:
- P1, P2: footprint w_pin_strip.pretty:pin_socket_2 -> P1P2_EDU_pin_strip_pretty:pin_strip_2mm_2
- XA1: footprint pf:Conn_Poncho_Derecha -> CESE_pretty:Conn_Poncho_Derecha
Changed lines of the file:
@@
 $EndComp
 $Comp
-L +3.3V #PWR01
+L +3.3V #PWR1
 U 1 1 596D4C32
 P 2300 2400
-F 0 "#PWR01" H 2300 2250 50  0001 C CNN
+F 0 "#PWR1" H 2300 2250 50  0001 C CNN
 F 1 "+3.3V" H 2300 2540 50  0000 C CNN
 F 2 "" H 2300 2400 50  0000 C CNN
@@
 $EndComp
 $Comp
-L GND #PWR02
+L GND #PWR3
 U 1 1 596D83A5
 P 3250 3000
-F 0 "#PWR02" H 3250 2750 50  0001 C CNN
+F 0 "#PWR3" H 3250 2750 50  0001 C CNN
 F 1 "GND" H 3150 2900 50  0000 C CNN
 F 2 "" H 3250 3000 50  0000 C CNN
@@
 $EndComp
 $Comp
-L GND #PWR03
+L GND #PWR4
 U 1 1 596D9266
 P 3300 2100
-F 0 "#PWR03" H 3300 1850 50  0001 C CNN
+F 0 "#PWR4" H 3300 1850 50  0001 C CNN
 F 1 "GND" H 3300 1950 50  0000 C CNN
 F 2 "" H 3300 2100 50  0000 C CNN
@@
 $EndComp
 $Comp
-L +5V #PWR04
+L +5V #PWR7
 U 1 1 596E40D8
 P 4150 1750
-F 0 "#PWR04" H 4150 1600 50  0001 C CNN
+F 0 "#PWR7" H 4150 1600 50  0001 C CNN
 F 1 "+5V" H 4150 1890 50  0000 C CNN
 F 2 "" H 4150 1750 50  0000 C CNN
@@
 D+
 $Comp
-L GND #PWR05
+L GND #PWR10
 U 1 1 596FB66D
 P 6200 3550
-F 0 "#PWR05" H 6200 3300 50  0001 C CNN
+F 0 "#PWR10" H 6200 3300 50  0001 C CNN
 F 1 "GND" H 6200 3400 50  0000 C CNN
 F 2 "" H 6200 3550 50  0000 C CNN
@@
 $EndComp
 $Comp
-L +5V #PWR06
+L +5V #PWR8
 U 1 1 5972BCCC
 P 4450 4500
-F 0 "#PWR06" H 4450 4350 50  0001 C CNN
+F 0 "#PWR8" H 4450 4350 50  0001 C CNN
 F 1 "+5V" H 4450 4640 50  0000 C CNN
 F 2 "" H 4450 4500 50  0000 C CNN
@@
 $EndComp
 $Comp
-L +3.3V #PWR07
+L +3.3V #PWR11
 U 1 1 5972BDCD
 P 6750 4550
-F 0 "#PWR07" H 6750 4400 50  0001 C CNN
+F 0 "#PWR11" H 6750 4400 50  0001 C CNN
 F 1 "+3.3V" H 6750 4690 50  0000 C CNN
 F 2 "" H 6750 4550 50  0000 C CNN
@@
 $EndComp
 $Comp
-L GND #PWR08
+L GND #PWR9
 U 1 1 59730224
 P 5200 4800
-F 0 "#PWR08" H 5200 4550 50  0001 C CNN
+F 0 "#PWR9" H 5200 4550 50  0001 C CNN
 F 1 "GND" H 5050 4750 50  0000 C CNN
 F 2 "" H 5200 4800 50  0000 C CNN
@@
 NoConn ~ 6200 4950
 $Comp
-L GND #PWR09
+L GND #PWR12
 U 1 1 59732AB0
 P 6900 4950
-F 0 "#PWR09" H 6900 4700 50  0001 C CNN
+F 0 "#PWR12" H 6900 4700 50  0001 C CNN
 F 1 "GND" H 6900 4800 50  0000 C CNN
 F 2 "" H 6900 4950 50  0000 C CNN
@@
 $EndComp
 $Comp
-L +5V #PWR010
+L +5V #PWR14
 U 1 1 597421A5
 P 9400 4200
-F 0 "#PWR010" H 9400 4050 50  0001 C CNN
+F 0 "#PWR14" H 9400 4050 50  0001 C CNN
 F 1 "+5V" H 9400 4340 50  0000 C CNN
 F 2 "" H 9400 4200 50  0000 C CNN
@@
 $EndComp
 $Comp
-L GND #PWR011
+L GND #PWR18
 U 1 1 59744849
 P 10300 3750
-F 0 "#PWR011" H 10300 3500 50  0001 C CNN
+F 0 "#PWR18" H 10300 3500 50  0001 C CNN
 F 1 "GND" H 10300 3600 50  0000 C CNN
 F 2 "" H 10300 3750 50  0000 C CNN
@@
 $EndComp
 $Comp
-L GND #PWR012
+L GND #PWR15
 U 1 1 5974491B
 P 9400 5200
-F 0 "#PWR012" H 9400 4950 50  0001 C CNN
+F 0 "#PWR15" H 9400 4950 50  0001 C CNN
 F 1 "GND" H 9400 5050 50  0000 C CNN
 F 2 "" H 9400 5200 50  0000 C CNN
@@
 $EndComp
 $Comp
-L GND #PWR013
+L GND #PWR19
 U 1 1 597449E6
 P 10650 3750
-F 0 "#PWR013" H 10650 3500 50  0001 C CNN
+F 0 "#PWR19" H 10650 3500 50  0001 C CNN
 F 1 "GND" H 10650 3600 50  0000 C CNN
 F 2 "" H 10650 3750 50  0000 C CNN
@@
 $EndComp
 $Comp
-L +3.3V #PWR014
+L +3.3V #PWR17
 U 1 1 5974E46F
 P 9550 2250
-F 0 "#PWR014" H 9550 2100 50  0001 C CNN
+F 0 "#PWR17" H 9550 2100 50  0001 C CNN
 F 1 "+3.3V" H 9550 2390 50  0000 C CNN
 F 2 "" H 9550 2250 50  0000 C CNN
@@
 F 0 "XA1" H 2950 5300 60  0000 C CNN
 F 1 "Conn_Poncho2P_2x_20x2" H 3000 3200 60  0000 C CNN
-F 2 "pf:Conn_Poncho_Derecha" H 2650 4900 60  0001 C CNN
+F 2 "CESE_pretty:Conn_Poncho_Derecha" H 2650 4900 60  0001 C CNN
 F 3 "" H 2650 4900 60  0000 C CNN
 F 4 "952-1938-ND" H 2650 4900 60  0001 C CNN "Digikey#"
@@
 NoConn ~ 8850 4550
 $Comp
-L PWR_FLAG #FLG015
+L PWR_FLAG #FLG1
 U 1 1 596C711A
 P 5150 4500
-F 0 "#FLG015" H 5150 4595 50  0001 C CNN
+F 0 "#FLG1" H 5150 4595 50  0001 C CNN
 F 1 "PWR_FLAG" H 5150 4680 50  0000 C CNN
 F 2 "" H 5150 4500 50  0000 C CNN
@@
 $EndComp
 $Comp
-L GND #PWR016
+L GND #PWR13
 U 1 1 5979E994
 P 9000 4750
-F 0 "#PWR016" H 9000 4500 50  0001 C CNN
+F 0 "#PWR13" H 9000 4500 50  0001 C CNN
 F 1 "GND" H 9000 4600 50  0000 C CNN
 F 2 "" H 9000 4750 50  0000 C CNN
@@
 $EndComp
 $Comp
-L GND #PWR017
+L GND #PWR16
 U 1 1 5979EBD6
 P 9450 3250
-F 0 "#PWR017" H 9450 3000 50  0001 C CNN
+F 0 "#PWR16" H 9450 3000 50  0001 C CNN
 F 1 "GND" H 9450 3100 50  0000 C CNN
 F 2 "" H 9450 3250 50  0000 C CNN
@@
 $EndComp
 $Comp
-L GND #PWR018
+L GND #PWR6
 U 1 1 5979ECDD
 P 3750 4700
-F 0 "#PWR018" H 3750 4450 50  0001 C CNN
+F 0 "#PWR6" H 3750 4450 50  0001 C CNN
 F 1 "GND" H 3750 4550 50  0000 C CNN
 F 2 "" H 3750 4700 50  0000 C CNN
@@
 NoConn ~ 3600 6200
 $Comp
-L +3.3V #PWR019
+L +3.3V #PWR2
 U 1 1 597BD5BA
 P 2350 4550
-F 0 "#PWR019" H 2350 4400 50  0001 C CNN
+F 0 "#PWR2" H 2350 4400 50  0001 C CNN
 F 1 "+3.3V" H 2350 4690 50  0000 C CNN
 F 2 "" H 2350 4550 50  0000 C CNN
@@
 $EndComp
 $Comp
-L +5V #PWR020
+L +5V #PWR5
 U 1 1 597BD8D9
 P 3650 4550
-F 0 "#PWR020" H 3650 4400 50  0001 C CNN
+F 0 "#PWR5" H 3650 4400 50  0001 C CNN
 F 1 "+5V" H 3650 4690 50  0000 C CNN
 F 2 "" H 3650 4550 50  0000 C CNN
@@
 F 0 "P1" H 4750 4500 50  0000 C CNN
 F 1 "CONN_01X02" V 4850 4350 50  0000 C CNN
-F 2 "w_pin_strip.pretty:pin_socket_2" H 4750 4350 50  0001 C CNN
+F 2 "P1P2_EDU_pin_strip_pretty:pin_strip_2mm_2" H 4750 4350 50  0001 C CNN
 F 3 "" H 4750 4350 50  0000 C CNN
 F 4 "952-1938-ND" H 4750 4350 60  0001 C CNN "Digikey#"
@@
 F 0 "P2" H 6350 4500 50  0000 C CNN
 F 1 "CONN_01X02" V 6450 4350 50  0000 C CNN
-F 2 "w_pin_strip.pretty:pin_socket_2" H 6350 4350 50  0001 C CNN
+F 2 "P1P2_EDU_pin_strip_pretty:pin_strip_2mm_2" H 6350 4350 50  0001 C CNN
 F 3 "" H 6350 4350 50  0000 C CNN
 F 4 "952-1938-ND" H 6350 4350 60  0001 C CNN "Digikey#"

Commit message: Imagen para el repositorio
Adjunto imagen para mejorar la presentación en el repositorio
Parts:
- U3: Digikey# 768-1129-1-ND -> 768-1128-2-ND; Manf# FT231XS-R -> FT231XQ-R
Changed lines of the file:
@@
 F 6 "Warning" H 4800 3150 50  0001 L BNN "Availability"
 F 7 "2.63 USD" H 4800 2950 50  0001 L BNN "Price_aprox"
-F 8 "768-1129-1-ND" H 5150 2650 60  0001 C CNN "Digikey#"
+F 8 "768-1128-2-ND" H 5150 2650 60  0001 C CNN "Digikey#"
 F 9 "FTDI, Future Technology Devices International Ltd" H 5150 2650 60  0001 C CNN "Manf"
-F 10 "FT231XS-R" H 5150 2650 60  0001 C CNN "Manf#"
+F 10 "FT231XQ-R" H 5150 2650 60  0001 C CNN "Manf#"
 	1    5150 2650
 	1    0    0    -1
@@
 $EndComp
 $Comp
-L +3.3V #PWR1
+L +3.3V #PWR01
 U 1 1 596D4C32
 P 2300 2400
-F 0 "#PWR1" H 2300 2250 50  0001 C CNN
+F 0 "#PWR01" H 2300 2250 50  0001 C CNN
 F 1 "+3.3V" H 2300 2540 50  0000 C CNN
 F 2 "" H 2300 2400 50  0000 C CNN
@@
 $EndComp
 $Comp
-L GND #PWR3
+L GND #PWR02
 U 1 1 596D83A5
 P 3250 3000
-F 0 "#PWR3" H 3250 2750 50  0001 C CNN
+F 0 "#PWR02" H 3250 2750 50  0001 C CNN
 F 1 "GND" H 3150 2900 50  0000 C CNN
 F 2 "" H 3250 3000 50  0000 C CNN
@@
 $EndComp
 $Comp
-L GND #PWR4
+L GND #PWR03
 U 1 1 596D9266
 P 3300 2100
-F 0 "#PWR4" H 3300 1850 50  0001 C CNN
+F 0 "#PWR03" H 3300 1850 50  0001 C CNN
 F 1 "GND" H 3300 1950 50  0000 C CNN
 F 2 "" H 3300 2100 50  0000 C CNN
@@
 $EndComp
 $Comp
-L +5V #PWR7
+L +5V #PWR04
 U 1 1 596E40D8
 P 4150 1750
-F 0 "#PWR7" H 4150 1600 50  0001 C CNN
+F 0 "#PWR04" H 4150 1600 50  0001 C CNN
 F 1 "+5V" H 4150 1890 50  0000 C CNN
 F 2 "" H 4150 1750 50  0000 C CNN
@@
 D+
 $Comp
-L GND #PWR10
+L GND #PWR05
 U 1 1 596FB66D
 P 6200 3550
-F 0 "#PWR10" H 6200 3300 50  0001 C CNN
+F 0 "#PWR05" H 6200 3300 50  0001 C CNN
 F 1 "GND" H 6200 3400 50  0000 C CNN
 F 2 "" H 6200 3550 50  0000 C CNN
@@
 $EndComp
 $Comp
-L +5V #PWR8
+L +5V #PWR06
 U 1 1 5972BCCC
 P 4450 4500
-F 0 "#PWR8" H 4450 4350 50  0001 C CNN
+F 0 "#PWR06" H 4450 4350 50  0001 C CNN
 F 1 "+5V" H 4450 4640 50  0000 C CNN
 F 2 "" H 4450 4500 50  0000 C CNN
@@
 $EndComp
 $Comp
-L +3.3V #PWR11
+L +3.3V #PWR07
 U 1 1 5972BDCD
 P 6750 4550
-F 0 "#PWR11" H 6750 4400 50  0001 C CNN
+F 0 "#PWR07" H 6750 4400 50  0001 C CNN
 F 1 "+3.3V" H 6750 4690 50  0000 C CNN
 F 2 "" H 6750 4550 50  0000 C CNN
@@
 $EndComp
 $Comp
-L GND #PWR9
+L GND #PWR08
 U 1 1 59730224
 P 5200 4800
-F 0 "#PWR9" H 5200 4550 50  0001 C CNN
+F 0 "#PWR08" H 5200 4550 50  0001 C CNN
 F 1 "GND" H 5050 4750 50  0000 C CNN
 F 2 "" H 5200 4800 50  0000 C CNN
@@
 NoConn ~ 6200 4950
 $Comp
-L GND #PWR12
+L GND #PWR09
 U 1 1 59732AB0
 P 6900 4950
-F 0 "#PWR12" H 6900 4700 50  0001 C CNN
+F 0 "#PWR09" H 6900 4700 50  0001 C CNN
 F 1 "GND" H 6900 4800 50  0000 C CNN
 F 2 "" H 6900 4950 50  0000 C CNN
@@
 $EndComp
 $Comp
-L +5V #PWR14
+L +5V #PWR010
 U 1 1 597421A5
 P 9400 4200
-F 0 "#PWR14" H 9400 4050 50  0001 C CNN
+F 0 "#PWR010" H 9400 4050 50  0001 C CNN
 F 1 "+5V" H 9400 4340 50  0000 C CNN
 F 2 "" H 9400 4200 50  0000 C CNN
@@
 $EndComp
 $Comp
-L GND #PWR18
+L GND #PWR011
 U 1 1 59744849
 P 10300 3750
-F 0 "#PWR18" H 10300 3500 50  0001 C CNN
+F 0 "#PWR011" H 10300 3500 50  0001 C CNN
 F 1 "GND" H 10300 3600 50  0000 C CNN
 F 2 "" H 10300 3750 50  0000 C CNN
@@
 $EndComp
 $Comp
-L GND #PWR15
+L GND #PWR012
 U 1 1 5974491B
 P 9400 5200
-F 0 "#PWR15" H 9400 4950 50  0001 C CNN
+F 0 "#PWR012" H 9400 4950 50  0001 C CNN
 F 1 "GND" H 9400 5050 50  0000 C CNN
 F 2 "" H 9400 5200 50  0000 C CNN
@@
 $EndComp
 $Comp
-L GND #PWR19
+L GND #PWR013
 U 1 1 597449E6
 P 10650 3750
-F 0 "#PWR19" H 10650 3500 50  0001 C CNN
+F 0 "#PWR013" H 10650 3500 50  0001 C CNN
 F 1 "GND" H 10650 3600 50  0000 C CNN
 F 2 "" H 10650 3750 50  0000 C CNN
@@
 $EndComp
 $Comp
-L +3.3V #PWR17
+L +3.3V #PWR014
 U 1 1 5974E46F
 P 9550 2250
-F 0 "#PWR17" H 9550 2100 50  0001 C CNN
+F 0 "#PWR014" H 9550 2100 50  0001 C CNN
 F 1 "+3.3V" H 9550 2390 50  0000 C CNN
 F 2 "" H 9550 2250 50  0000 C CNN
@@
 NoConn ~ 8850 4550
 $Comp
-L PWR_FLAG #FLG1
+L PWR_FLAG #FLG015
 U 1 1 596C711A
 P 5150 4500
-F 0 "#FLG1" H 5150 4595 50  0001 C CNN
+F 0 "#FLG015" H 5150 4595 50  0001 C CNN
 F 1 "PWR_FLAG" H 5150 4680 50  0000 C CNN
 F 2 "" H 5150 4500 50  0000 C CNN
@@
 $EndComp
 $Comp
-L GND #PWR13
+L GND #PWR016
 U 1 1 5979E994
 P 9000 4750
-F 0 "#PWR13" H 9000 4500 50  0001 C CNN
+F 0 "#PWR016" H 9000 4500 50  0001 C CNN
 F 1 "GND" H 9000 4600 50  0000 C CNN
 F 2 "" H 9000 4750 50  0000 C CNN
@@
 $EndComp
 $Comp
-L GND #PWR16
+L GND #PWR017
 U 1 1 5979EBD6
 P 9450 3250
-F 0 "#PWR16" H 9450 3000 50  0001 C CNN
+F 0 "#PWR017" H 9450 3000 50  0001 C CNN
 F 1 "GND" H 9450 3100 50  0000 C CNN
 F 2 "" H 9450 3250 50  0000 C CNN
@@
 $EndComp
 $Comp
-L GND #PWR6
+L GND #PWR018
 U 1 1 5979ECDD
 P 3750 4700
-F 0 "#PWR6" H 3750 4450 50  0001 C CNN
+F 0 "#PWR018" H 3750 4450 50  0001 C CNN
 F 1 "GND" H 3750 4550 50  0000 C CNN
 F 2 "" H 3750 4700 50  0000 C CNN
@@
 NoConn ~ 3600 6200
 $Comp
-L +3.3V #PWR2
+L +3.3V #PWR019
 U 1 1 597BD5BA
 P 2350 4550
-F 0 "#PWR2" H 2350 4400 50  0001 C CNN
+F 0 "#PWR019" H 2350 4400 50  0001 C CNN
 F 1 "+3.3V" H 2350 4690 50  0000 C CNN
 F 2 "" H 2350 4550 50  0000 C CNN
@@
 $EndComp
 $Comp
-L +5V #PWR5
+L +5V #PWR020
 U 1 1 597BD8D9
 P 3650 4550
-F 0 "#PWR5" H 3650 4400 50  0001 C CNN
+F 0 "#PWR020" H 3650 4400 50  0001 C CNN
 F 1 "+5V" H 3650 4690 50  0000 C CNN
 F 2 "" H 3650 4550 50  0000 C CNN

Commit message: Actualización 33Ohm
Actualización de la resistencia de 330 Ohm para el usos de Kicost
Parts:
- R5: Digikey# (none) -> RMCF0603JT330RCT-ND; Manf (none) -> Stackpole Electronics Inc.; Manf# (none) -> RMCF0603JT330R
Changed lines of the file:
@@
 F 2 "Resistors_SMD:R_0603_HandSoldering" V 10230 2950 50  0001 C CNN
 F 3 "" H 10300 2950 50  0000 C CNN
+F 4 "RMCF0603JT330RCT-ND" V 10300 2950 60  0001 C CNN "Digikey#"
+F 5 "Stackpole Electronics Inc." V 10300 2950 60  0001 C CNN "Manf"
+F 6 "RMCF0603JT330R" V 10300 2950 60  0001 C CNN "Manf#"
 	1    10300 2950
 	-1   0    0    -1
